File: hardware/Automatic Watering System/Automatic Watering System.kicad_pcb (KiCad board)
At the start: 2 copper layers, 14 parts, among them J1 LC709203 Board, J2 Conn_01x05_Socket, J5 SEN0193 Analog Capacitive Soi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, U1 DHT11, U2 TP4056

Commit message: edits to documents
Parts:
- removed U2: TP4056, Package_SO:SOIC-8_3.9x4.9mm_P1.27mm
- added REF**: MountingHole_4.3mm_M4, MountingHole:MountingHole_4.3mm_M4, F.Cu at (42.8, 129.3)
- added REF**: MountingHole_4.3mm_M4, MountingHole:MountingHole_4.3mm_M4, F.Cu at (113.2, 129.0)
- added U3: TP4056 Li-Po Battery Charger Module, Power Management:TP4056 1A Li-ion Battery Charging Module, F.Cu at (92.4, 149.2)
- D1: value LED_RGBA -> STATUS_LED
- J2: value Conn_01x05_Socket -> Ambient Light Sensor
- J5: value SEN0193 Analog Capacitive Soil Moisture Sensor -> Soil Moisture Sensor
- moved D2 108.1 mm to (214.7, 56.0)
- moved J1 95.1 mm to (81.0, 136.2), turned to -90 degrees
- moved D1 74.5 mm to (110.0, 110.5), turned to 0 degrees
- moved SC1 71.2 mm to (195.0, 57.8)
- moved R1 69.1 mm to (207.7, 68.8)
- moved U1 67.5 mm to (58.4, 101.5), turned to 90 degrees
- moved R2 65.7 mm to (202.4, 78.0)
- moved R3 65.7 mm to (202.4, 81.2)
- moved R4 65.7 mm to (202.4, 84.3)
- moved BT1 64.6 mm to (185.0, 90.4)
- moved J5 53.3 mm to (97.0, 100.2), turned to -90 degrees
- moved A1 52.8 mm to (77.5, 120.4), turned to -90 degrees
- moved J2 44.8 mm to (75.3, 100.5), turned to 90 degrees
Connections:
- BT1 pad GND: GND -> (no net)
- J1 pad 1: VIN -> BATTERY_MON(+)
- J1 pad 2: GND -> BATTERY_MON(-)
Routing:
- net BATTERY_MON(+): track 0.00 -> 32.7 mm
- net BATTERY_MON_SDA: track 0.00 -> 4.78 mm
- net BATTERY_MON_SCL: track 0.00 -> 4.78 mm
- net BATTERY_MON_INT: track 0.00 -> 4.78 mm
Other:
- board outline added: 94.9 x 65.8 mm
