File: hardware/Automatic Watering System/Automatic Watering System.kicad_sch (KiCad schematic)
At the start: 14 parts, among them J1 LC709203 Board, J2 Conn_01x05_Socket, J5 SEN0193 Analog Capacitive Soi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, U1 DHT11, U2 TP4056

Commit message: edits to documents
Parts:
- removed R4: 1.2k, Resistor_THT:R_Axial_DIN0204_L3.6mm_D1.6mm_P7.62mm_Horizontal, symbol Device:R
- removed U2: TP4056, Package_SO:SOIC-8_3.9x4.9mm_P1.27mm, symbol TP4056:TP4056
- added U3: TP4056 Li-Po Battery Charger Module, Power Management:TP4056 1A Li-ion Battery Charging Module, symbol Battery_Management:TP4056_Lipo_Battery_Charging_Board_Module
- D1: value LED_RGBA -> STATUS_LED
- J2: value Conn_01x05_Socket -> Ambient Light Sensor
- J5: value SEN0193 Analog Capacitive Soil Moisture Sensor -> Soil Moisture Sensor
Connections:
- net VIN is gone; now on net BATTERY_MON(+): J1.1 (Pin_1)
- net BATTERY_MON(+): now also U3.3 (IN+)
- net BATTERY_MON(-): now also J1.2 (Pin_2), U3.4 (IN-)
- net GND: now also U3.2 (BAT-); no longer J1.2 (Pin_2)
- net at D2.1 (K): now also U3.1 (BAT+)
- no-connect marks 13 -> 11
